File: Bottle_PCB.brd (EAGLE design)
At the start: 100 x 50 mm, 81 parts, among them J1 GROVE-4P-2.0-SMD, Q1 8.000 MHz, Q5 ZVN 3306 F, Q6 ZVN 3306 F, Q7 ZVN 3306 F, U1 USD-SOCKETNEW

Commit message: - employed several more libraries from Seed Studio and Arduino Project - replaced power supply with modern solution, charging circuitry etc.
Parts:
- removed C_U12V: 100µF/16V, _E:SMC_D
- removed C_U5V: 100µF/6,3V, _E:SMC_D
- removed D_U5V: MBRS120, _D:SMB
- removed LM2594_3.3: LM2594, _Voltage_Regulators:SO08
- removed L_U5V: 100µH, _Trafo_Spule:PISM
- removed R_U12V: 10k, quantum-sensor:R0805
- removed SV2, SV3: (no value), con-ml:ML10L
- removed T_U12V: (no value), _transistor:SOT23
- removed VIN: AK350/2, con-ptr500:AK350/2
- added C13: 1µF, rcl:C0805
- added C14, C15: 100nF, resistor:C0603
- added C_3V3, C_VIN, C_V_LIPO_USB: 10µ/10V, _E:SMC_D
- added D2, D3, D4: MSS1P2U, Seed-Discrete:D1005
- added IC1: LP2985-33DBV, Arduino-SmartPrj:SOT23-DBV
- added LED1: CHRG_Red, led:CHIPLED_0603
- added LED2: DONE_Green, led:CHIPLED_0603
- added LIPO-BAT, SOLAR: (no value), Seed-Battery-Connector:JST-2.0
- added R1, R16: 10k, rcl:R0603
- added R17: 330 (20mA) or 2k, rcl:R0603
- added R18, R19: 2M_1%, rcl:R0603
- added R20, R21: 10M_1%, rcl:R0603
- added SW_CHARGE_INDICATORS: (no value), switch-omron:B3F-10XX
- added T_LIPO_USB: (no value), _transistor:SOT23
- added U3: CN3065-1320040P1, OPL:DFN8
- added UART1_C1: 10n, Arduino-SmartPrj:C0603-ROUND
- R10: value 40k -> 10k; device rcl:M1206 -> rcl:R0603
- R11: device rcl:M1206 -> rcl:R0603
- SJ2, SJ4: device jumper:SJ -> jumper:SJ_2
- UART1_C10, UART1_C11, UART1_C2: device _C:C0805 -> Arduino-SmartPrj:C0603-ROUND
- UART1_RX_LED, UART1_TX_LED: device led:CHIPLED_0805 -> led:CHIPLED_0603
- moved R11 281.9 mm to (-68.0, -239.0), flipped to the top, turned to 0 degrees
- moved R10 281.7 mm to (-68.0, -234.0), flipped to the top, turned to 0 degrees
- moved SJ2 70.0 mm to (-46.0, -201.0)
- moved SJ4 67.0 mm to (-46.0, -206.0)
Connections:
- net PB2_VBATT_AIN0 renamed PB2_AIN0
- net PB3_VBATT_AIN1 renamed PB3_AIN1
- removed net N$16: SJ1.2, U2.1
- removed net N$17: SJ2.2, U2.2
- removed net N$19: SJ3.2, U2.3
- removed net N$21: SJ5.2, U2.9
- removed net N$24: SJ8.2, U2.11
- removed net N$25: SJ6.2, U2.15
- removed net N$26: SJ7.2, U2.16
- removed net PA4: AD.5, ATMEGA1284.33
- removed net PA5: AD.6, ATMEGA1284.32
- removed net SWITCH_OUT: D_U5V.C, LM2594_3.3.8, L_U5V.1
- removed net VBATT: R10.2, R11.1
- new net N$22: R1.2, U3.2
- new net N$27: U3.HEAT
- new net PA4_V_SOLAR: AD.5, ATMEGA1284.33, R19.1, R21.2
- new net PA5_V_LIPO: AD.6, ATMEGA1284.32, C14.2, C15.1, R18.1, R20.2
- new net PC4_!DONE: ATMEGA1284.23, LED2.C, R11.1, U3.6
- new net PC5_!CHRG: ATMEGA1284.24, LED1.C, R10.1, U3.7
- new net V_LIPO: C13.2, LIPO-BAT.1, R20.1, T_LIPO_USB.2, U3.5, U3.8
- new net V_LIPO_USB: C_V_LIPO_USB.+, D4.-, IC1.1, IC1.3, SW_CHARGE_INDICATORS.3, SW_CHARGE_INDICATORS.4, T_LIPO_USB.3
- new net V_SOLAR: D2.+, SOLAR.1
- net +3V3: now also C_3V3.+, IC1.5, R10.2, R11.2; no longer C_U5V.+, LM2594_3.3.4, L_U5V.2, R2.1, SV2.1, SV2.3, SV3.1, SV3.3
- net +5V: now also D3.+, D4.+, R16.2, T_LIPO_USB.1
- net BEE_RESET: now also SJ8.2, U2.11
- net BEE_STATUS: now also SJ6.2, U2.15
- net BEE_VCC: now also SJ5.2, U2.9
- net FTDI_CTS: now also SJ3.2, U2.3
- net FTDI_DTR: now also SJ7.2, U2.16
- net FTDI_RTS: now also SJ1.2, U2.1
- net GND: now also C13.1, C14.1, C15.2, C_3V3.-, C_VIN.-, C_V_LIPO_USB.-, IC1.2, LIPO-BAT.2, R1.1, R16.1, R18.2, R19.2, SOLAR.2, U3.1, U3.3, UART1_C1.2; no longer C_U12V.-, C_U5V.-, D_U5V.A, LM2594_3.3.5, LM2594_3.3.6, R11.2, R_U12V.2, SV2.2, SV2.4, SV2.6, SV3.2, SV3.4, SV3.6, VIN.P$1
- net N$18: now also LED1.A, LED2.A, R17.1; no longer R_U12V.1, T_U12V.1
- net N$20: now also R17.2, SW_CHARGE_INDICATORS.1, SW_CHARGE_INDICATORS.2; no longer SJ4.2, U2.4
- net N$3: now also IC1.4, UART1_C1.1; no longer T_U12V.2, VIN.P$2
- net N$31: now also R2.1
- net PD0_RXD0_USB: now also SJ2.2, SJ4.3, U2.2
- net PD1_TXD0_USB: now also SJ2.3, SJ4.2, U2.4
- net VIN: now also C_VIN.+, D2.-, D3.-, R21.1, U3.4; no longer C_U12V.+, LM2594_3.3.7, R10.1, SV2.9, SV3.9, T_U12V.3
Routing:
- net GND: track 417.1 -> 331.2 mm
- net VIN: track 63.6 -> 0.00 mm, vias 2 -> 0
- net +3V3: track 321.2 -> 266.4 mm, vias 11 -> 10
- net VBATT: track 34.2 -> 0.00 mm, vias 3 -> 0
- net SWITCH_OUT: track 16.6 -> 0.00 mm, vias 1 -> 0
- net N$18: track 4.05 -> 0.00 mm
- net N$3: track 3.54 -> 0.00 mm
